File: pcb/ultra-choc-wings.kicad_pcb (KiCad board)
At the start: 2 copper layers, 110.3 x 90.1 mm, 84 parts, among them Q1 AO3400A, SW1 CPG1316S01D02_reversible, SW10 CPG1316S01D02_reversible, SW11 CPG1316S01D02_reversible, SW12 CPG1316S01D02_reversible, SW13 CPG1316S01D02_reversible, SW14 CPG1316S01D02_reversible, SW15 CPG1316S01D02_reversible, SW16 CPG1316S01D02_reversible, SW17 CPG1316S01D02_reversible, SW18 CPG1316S01D02_reversible, SW2 CPG1316S01D02_reversible, SW3 CPG1316S01D02_reversible, SW4 CPG1316S01D02_reversible, SW5 CPG1316S01D02_reversible, SW6 CPG1316S01D02_reversible, SW7 CPG1316S01D02_reversible, SW8 CPG1316S01D02_reversible, SW9 CPG1316S01D02_reversible

Commit message: fix(update): update the kicad version
Parts:
- moved D1 234.1 mm to (170.9, 169.9)
- moved D10 234.1 mm to (224.9, 158.5)
- moved D11 234.1 mm to (224.9, 141.5)
- moved D12 234.1 mm to (224.9, 124.5)
- moved D13 234.1 mm to (242.9, 160.9)
- moved D14 234.1 mm to (242.9, 143.9)
- moved D15 234.1 mm to (242.9, 126.9)
- moved D16 234.1 mm to (217.7, 164.1)
- moved D17 234.1 mm to (239.6, 167.3)
- moved D2 234.1 mm to (170.9, 152.9)
- moved D3 234.1 mm to (170.9, 135.9)
- moved D4 234.1 mm to (188.9, 157.9)
- moved D5 234.1 mm to (188.9, 140.9)
- moved D6 234.1 mm to (188.9, 123.9)
- moved D7 234.1 mm to (206.9, 151.9)
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