File: pcb/ultra-choc-wings.kicad_pcb (KiCad board)
At the start: 2 copper layers, 110.3 x 90.1 mm, 84 parts, among them Q1 AO3400A, SW1 CPG1316S01D02_reversible, SW10 CPG1316S01D02_reversible, SW11 CPG1316S01D02_reversible, SW12 CPG1316S01D02_reversible, SW13 CPG1316S01D02_reversible, SW14 CPG1316S01D02_reversible, SW15 CPG1316S01D02_reversible, SW16 CPG1316S01D02_reversible, SW17 CPG1316S01D02_reversible, SW18 CPG1316S01D02_reversible, SW2 CPG1316S01D02_reversible, SW3 CPG1316S01D02_reversible, SW4 CPG1316S01D02_reversible, SW5 CPG1316S01D02_reversible, SW6 CPG1316S01D02_reversible, SW7 CPG1316S01D02_reversible, SW8 CPG1316S01D02_reversible, SW9 CPG1316S01D02_reversible

Commit message: Link the board footprints to the ucw library and the schematic
Each footprint now names its ucw library footprint and carries the path of
its schematic symbol, so cross-probing and Update PCB from Schematic match
part for part. Text-only edit of the KiCad 10 board; nothing moved.

Co-Authored-By: Claude Opus 5.5 (1M context) <noreply@anthropic.com>
Claude-Session: https://claude.ai/code/session_0165D9fBjcdWGjdLPuN9BjoD
Parts:
- PAD1: footprint SMDPad -> ucw:SMDPad
- SW1, SW10, SW11, SW12, SW13, SW14, SW15, SW16, SW17, SW18, SW2, SW3, SW4, SW5, SW6, SW7, SW8, SW9: footprint CPG1316S01D02_reversible -> ucw:CPG1316S01D02_reversible
- xiao-ble1: footprint xiao-ble -> ucw:xiao-ble
Changed lines of the file:
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@@
 		(embedded_fonts no)
 	)
-	(footprint "CPG1316S01D02_reversible"
+	(footprint "ucw:CPG1316S01D02_reversible"
 		(layer "F.Cu")
 		(at 222.2968 151.3218)
@@
 		(embedded_fonts no)
 	)
-	(footprint "CPG1316S01D02_reversible"
+	(footprint "ucw:CPG1316S01D02_reversible"
 		(layer "F.Cu")
 		(at 222.2968 134.3218)
@@
 		(embedded_fonts no)
 	)
-	(footprint "SMDPad"
+	(footprint "ucw:SMDPad"
 		(layer "F.Cu")
 		(at 168.2968 120.1968)
@@
 		(embedded_fonts no)
 	)
-	(footprint "CPG1316S01D02_reversible"
+	(footprint "ucw:CPG1316S01D02_reversible"
 		(layer "F.Cu")
 		(at 168.2968 162.6968)
@@
 		(embedded_fonts no)
 	)
-	(footprint "CPG1316S01D02_reversible"
+	(footprint "ucw:CPG1316S01D02_reversible"
 		(layer "F.Cu")
 		(at 186.2968 116.6968)
@@
 		(embedded_fonts no)
 	)
-	(footprint "CPG1316S01D02_reversible"
+	(footprint "ucw:CPG1316S01D02_reversible"
 		(layer "F.Cu")
 		(at 222.2968 117.3218)
@@
 		(embedded_fonts no)
 	)
-	(footprint "CPG1316S01D02_reversible"
+	(footprint "ucw:CPG1316S01D02_reversible"
 		(layer "F.Cu")
 		(at 240.2968 119.6968)
@@
 		(embedded_fonts no)
 	)
-	(footprint "CPG1316S01D02_reversible"
+	(footprint "ucw:CPG1316S01D02_reversible"
 		(layer "F.Cu")
 		(at 186.2968 133.6968)
@@
 		(embedded_fonts no)
 	)
-	(footprint "CPG1316S01D02_reversible"
+	(footprint "ucw:CPG1316S01D02_reversible"
 		(layer "F.Cu")
 		(at 186.2968 150.6968)
@@
 		(embedded_fonts no)
 	)
-	(footprint "CPG1316S01D02_reversible"
+	(footprint "ucw:CPG1316S01D02_reversible"
 		(layer "F.Cu")
 		(at 168.2968 145.6968)
@@
 		(embedded_fonts no)
 	)
-	(footprint "CPG1316S01D02_reversible"
+	(footprint "ucw:CPG1316S01D02_reversible"
 		(layer "F.Cu")
 		(at 236.4468 173.8768 -15)
@@
 		(embedded_fonts no)
 	)
-	(footprint "CPG1316S01D02_reversible"
+	(footprint "ucw:CPG1316S01D02_reversible"
 		(layer "F.Cu")
 		(at 204.2968 127.6968)
@@
 		(embedded_fonts no)
 	)
-	(footprint "CPG1316S01D02_reversible"
+	(footprint "ucw:CPG1316S01D02_reversible"
 		(layer "F.Cu")
 		(at 240.2968 136.6968)
@@
 		(embedded_fonts no)
 	)
-	(footprint "CPG1316S01D02_reversible"
+	(footprint "ucw:CPG1316S01D02_reversible"
 		(layer "F.Cu")
 		(at 204.2968 144.6968)
@@
 		(embedded_fonts no)
 	)
-	(footprint "CPG1316S01D02_reversible"
+	(footprint "ucw:CPG1316S01D02_reversible"
 		(layer "F.Cu")
 		(at 168.2968 128.6968)
@@
 		(embedded_fonts no)
 	)
-	(footprint "CPG1316S01D02_reversible"
+	(footprint "ucw:CPG1316S01D02_reversible"
 		(layer "F.Cu")
 		(at 204.2968 110.6968)
@@
 		(embedded_fonts no)
 	)
-	(footprint "xiao-ble"
+	(footprint "ucw:xiao-ble"
 		(layer "F.Cu")
 		(at 159.4068 119.6968 -90)
@@
 		(embedded_fonts no)
 	)
-	(footprint "CPG1316S01D02_reversible"
+	(footprint "ucw:CPG1316S01D02_reversible"
 		(layer "F.Cu")
 		(at 216.3968 171.2868)
@@
 		(embedded_fonts no)
 	)
-	(footprint "CPG1316S01D02_reversible"
+	(footprint "ucw:CPG1316S01D02_reversible"
 		(layer "F.Cu")
 		(at 257.0468 177.0868 -30)
@@
 		(embedded_fonts no)
 	)
-	(footprint "CPG1316S01D02_reversible"
+	(footprint "ucw:CPG1316S01D02_reversible"
 		(layer "F.Cu")
 		(at 240.2968 153.6968)
