File: pcb/ultra-choc-wings.kicad_pcb (KiCad board)
At the start: 2 copper layers, 110.3 x 90.1 mm, 84 parts, among them Q1 AO3400A, SW1 CPG1316S01D02_reversible, SW10 CPG1316S01D02_reversible, SW11 CPG1316S01D02_reversible, SW12 CPG1316S01D02_reversible, SW13 CPG1316S01D02_reversible, SW14 CPG1316S01D02_reversible, SW15 CPG1316S01D02_reversible, SW16 CPG1316S01D02_reversible, SW17 CPG1316S01D02_reversible, SW18 CPG1316S01D02_reversible, SW2 CPG1316S01D02_reversible, SW3 CPG1316S01D02_reversible, SW4 CPG1316S01D02_reversible, SW5 CPG1316S01D02_reversible, SW6 CPG1316S01D02_reversible, SW7 CPG1316S01D02_reversible, SW8 CPG1316S01D02_reversible, SW9 CPG1316S01D02_reversible

Commit message: Re-route the board with the parts under the switches
Parts:
- moved D1 239.5 mm to (-2.90, 5.10)
- moved D10 239.5 mm to (51.1, -6.28)
- moved D11 239.5 mm to (51.1, -23.3)
- moved D12 239.5 mm to (51.1, -40.3)
- moved D13 239.5 mm to (69.1, -3.90)
- moved D14 239.5 mm to (69.1, -20.9)
- moved D15 239.5 mm to (69.1, -37.9)
- moved D2 239.5 mm to (-2.90, -11.9)
- moved D3 239.5 mm to (-2.90, -28.9)
- moved D4 239.5 mm to (15.1, -6.90)
- moved D5 239.5 mm to (15.1, -23.9)
- moved D6 239.5 mm to (15.1, -40.9)
- moved D7 239.5 mm to (33.1, -12.9)
- moved D8 239.5 mm to (33.1, -29.9)
- moved D9 239.5 mm to (33.1, -46.9)
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Routing:
- net LED_K: track 563.1 -> 471.6 mm, vias 15 -> 17
- net P4: track 149.9 -> 187.9 mm, vias 7 -> 5
- net middle_thumb: track 27.4 -> 9.77 mm
- net P1: track 148.3 -> 165.2 mm, vias 6 -> 5
- net LA_inner_bottom: track 36.3 -> 19.5 mm
- net VCC3: track 475.1 -> 489.2 mm, vias 17 -> 21
- net inner_thumb: track 22.7 -> 9.00 mm
- net ring_bottom: track 22.2 -> 8.63 mm
- net home_thumb: track 19.7 -> 8.09 mm, vias 2 -> 1
- net LA_ring_home: track 26.6 -> 16.4 mm, vias 1 -> 2
- net LA_ring_top: track 15.6 -> 25.1 mm
- net LA_pinky_bottom: track 27.0 -> 18.0 mm, vias 1 -> 3
- net P0: track 166.7 -> 175.6 mm
- net LA_index_home: track 27.0 -> 18.2 mm, vias 1 -> 2
- net LA_pinky_top: track 23.4 -> 14.7 mm, vias 1 -> 2
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