File: pcb/ultra-choc-wings.kicad_pcb (KiCad board)
At the start: 2 copper layers, 110.3 x 90.1 mm, 84 parts, among them Q1 AO3400A, SW1 CPG1316S01D02_reversible, SW10 CPG1316S01D02_reversible, SW11 CPG1316S01D02_reversible, SW12 CPG1316S01D02_reversible, SW13 CPG1316S01D02_reversible, SW14 CPG1316S01D02_reversible, SW15 CPG1316S01D02_reversible, SW16 CPG1316S01D02_reversible, SW17 CPG1316S01D02_reversible, SW18 CPG1316S01D02_reversible, SW2 CPG1316S01D02_reversible, SW3 CPG1316S01D02_reversible, SW4 CPG1316S01D02_reversible, SW5 CPG1316S01D02_reversible, SW6 CPG1316S01D02_reversible, SW7 CPG1316S01D02_reversible, SW8 CPG1316S01D02_reversible, SW9 CPG1316S01D02_reversible

Commit message: Re-route the board with the diode next to the LED
Co-Authored-By: Claude Sonnet 5.5 <noreply@anthropic.com>
Claude-Session: https://claude.ai/code/session_0165D9fBjcdWGjdLPuN9BjoD
Parts:
- D1, D10, D11, D12, D13, D14, D15, D16, D17, D18, D2, D3, D4, D5, D6, D7, D8, D9: value 1N4148W -> 1N4148WS; footprint ucw:REV_SOD123 -> ucw:REV_SOD323
- moved D18 7.48 mm to (89.7, 12.8)
- moved D14 7.48 mm to (72.0, -27.8)
- moved D13 7.48 mm to (72.0, -10.8)
- moved D11 7.48 mm to (54.0, -30.2)
- moved D5 7.48 mm to (18.0, -30.8)
- moved D15 7.48 mm to (72.0, -44.8)
- moved D10 7.48 mm to (54.0, -13.2)
- moved D2 7.48 mm to (0.00, -18.8)
- moved D3 7.48 mm to (0.00, -35.8)
- moved D4 7.48 mm to (18.0, -13.8)
- moved D6 7.48 mm to (18.0, -47.8)
- moved D7 7.48 mm to (36.0, -19.8)
- moved D1 7.48 mm to (0.00, -1.80)
- moved D16 7.48 mm to (48.1, 6.79)
- moved D12 7.48 mm to (54.0, -47.2)
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Routing:
- net P4: track 187.9 -> 156.2 mm, vias 5 -> 10
- net GND: track 152.1 -> 181.0 mm
- net P8: track 133.7 -> 117.7 mm
- net LA_index_home: track 18.2 -> 31.5 mm
- net P1: track 165.2 -> 176.7 mm, vias 5 -> 8
- net LA_index_top: track 14.8 -> 26.0 mm, vias 2 -> 1
- net SW_BAT: track 68.8 -> 58.4 mm
- net LA_pinky_top: track 14.7 -> 24.6 mm, vias 2 -> 1
- net LA_inner_top: track 14.8 -> 24.3 mm, vias 2 -> 1
- net LA_ring_home: track 16.4 -> 24.7 mm, vias 2 -> 1
- net LA_inner_thumb: track 15.4 -> 23.1 mm, vias 2 -> 1
- net middle_bottom: track 9.21 -> 16.7 mm
- net P2: track 137.3 -> 130.1 mm
- net LED_K: track 471.6 -> 464.5 mm, vias 17 -> 15
- net index_home: track 8.36 -> 13.4 mm
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