File: pcb/ultra-choc-wings.kicad_pcb (KiCad board)
At the start: 2 copper layers, 110.3 x 90.1 mm, 84 parts, among them Q1 AO3400A, SW1 CPG1316S01D02_reversible, SW10 CPG1316S01D02_reversible, SW11 CPG1316S01D02_reversible, SW12 CPG1316S01D02_reversible, SW13 CPG1316S01D02_reversible, SW14 CPG1316S01D02_reversible, SW15 CPG1316S01D02_reversible, SW16 CPG1316S01D02_reversible, SW17 CPG1316S01D02_reversible, SW18 CPG1316S01D02_reversible, SW2 CPG1316S01D02_reversible, SW3 CPG1316S01D02_reversible, SW4 CPG1316S01D02_reversible, SW5 CPG1316S01D02_reversible, SW6 CPG1316S01D02_reversible, SW7 CPG1316S01D02_reversible, SW8 CPG1316S01D02_reversible, SW9 CPG1316S01D02_reversible

Commit message: feat(render): add 3d model
Parts:
- SW1, SW10, SW11, SW12, SW13, SW14, SW15, SW16, SW17, SW18, SW2, SW3, SW4, SW5, SW6, SW7, SW8, SW9: value CPG1316S01D02_reversible -> CPG1316S01D02_reversible_mikefives; footprint ucw:CPG1316S01D02_reversible -> leptiosis:CPG1316S01D02_reversible_mikefives
- moved D16 233.9 mm to (219.6, 165.9)
- moved D18 233.9 mm to (261.1, 172.0)
- moved L16 233.9 mm to (219.6, 164.5)
- moved R16 233.9 mm to (219.6, 172.8)
- moved SW16 233.9 mm to (219.6, 167.7)
- moved BT1 233.9 mm to (193.4, 169.1)
- moved C1 233.9 mm to (200.4, 153.6)
- moved C2 233.9 mm to (204.4, 156.1)
- moved D1 233.9 mm to (171.4, 157.3)
- moved D10 233.9 mm to (225.4, 145.9)
- moved D11 233.9 mm to (225.4, 128.9)
- moved D12 233.9 mm to (225.4, 112.0)
- moved D13 233.9 mm to (243.4, 148.3)
- moved D14 233.9 mm to (243.4, 131.3)
- moved D15 233.9 mm to (243.4, 114.3)
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