File: pcb/ultra-choc-wings.kicad_sch (KiCad schematic)
At the start: 84 parts, among them Q1 AO3400A, SW1 CPG1316S01D02_reversible, SW10 CPG1316S01D02_reversible, SW11 CPG1316S01D02_reversible, SW12 CPG1316S01D02_reversible, SW13 CPG1316S01D02_reversible, SW14 CPG1316S01D02_reversible, SW15 CPG1316S01D02_reversible, SW16 CPG1316S01D02_reversible, SW17 CPG1316S01D02_reversible, SW18 CPG1316S01D02_reversible, SW2 CPG1316S01D02_reversible, SW3 CPG1316S01D02_reversible, SW4 CPG1316S01D02_reversible, SW5 CPG1316S01D02_reversible, SW6 CPG1316S01D02_reversible, SW7 CPG1316S01D02_reversible, SW8 CPG1316S01D02_reversible, SW9 CPG1316S01D02_reversible, T1 SPDT

Commit message: Refresh schematic links, libraries and 3D previews
Co-Authored-By: Claude Sonnet 5.5 <noreply@anthropic.com>
Claude-Session: https://claude.ai/code/session_0165D9fBjcdWGjdLPuN9BjoD
Parts:
- D1, D10, D11, D12, D13, D14, D15, D16, D17, D18, D2, D3, D4, D5, D6, D7, D8, D9: value 1N4148W -> 1N4148WS; footprint ucw:REV_SOD123 -> ucw:REV_SOD323; LCSC C81598 -> C2128
