File: output/pcbs/main.kicad_pcb (KiCad board)
At the start: 2 copper layers, 110.3 x 90.1 mm, 84 parts, among them Q1 AO3400A, SW1 CPG1316S01D02_reversible, SW10 CPG1316S01D02_reversible, SW11 CPG1316S01D02_reversible, SW12 CPG1316S01D02_reversible, SW13 CPG1316S01D02_reversible, SW14 CPG1316S01D02_reversible, SW15 CPG1316S01D02_reversible, SW16 CPG1316S01D02_reversible, SW17 CPG1316S01D02_reversible, SW18 CPG1316S01D02_reversible, SW2 CPG1316S01D02_reversible, SW3 CPG1316S01D02_reversible, SW4 CPG1316S01D02_reversible, SW5 CPG1316S01D02_reversible, SW6 CPG1316S01D02_reversible, SW7 CPG1316S01D02_reversible, SW8 CPG1316S01D02_reversible, SW9 CPG1316S01D02_reversible

Commit message: Re-route the board with the parts under the switches
Parts:
- moved R18 13.8 mm to (88.3, 20.0)
- moved R16 13.8 mm to (50.5, 13.7)
- moved R17 13.8 mm to (69.1, 16.7)
- moved D18 13.0 mm to (83.7, 17.4)
- moved D17 13.0 mm to (64.0, 15.4)
- moved D16 13.0 mm to (45.2, 13.7)
- moved D6 5.89 mm to (15.1, -40.9)
- moved D4 5.89 mm to (15.1, -6.90)
- moved D5 5.89 mm to (15.1, -23.9)
- moved D12 5.89 mm to (51.1, -40.3)
- moved D15 5.89 mm to (69.1, -37.9)
- moved D9 5.89 mm to (33.1, -46.9)
- moved D1 5.89 mm to (-2.90, 5.10)
- moved D10 5.89 mm to (51.1, -6.28)
- moved D11 5.89 mm to (51.1, -23.3)
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